Commit message: make ranger easy use

File: ranger_description/urdf/ranger_mini3_v3_simple.urdf (robot description, URDF)
Before this commit: robot ranger_mini_v3_simple, 9 links, 8 joints
Links:
- link base_link: mass 10 -> None
- link fl_steering_wheel_link: mass 1 -> None
- link fl_wheel_link: mass 8 -> None
- link fr_steering_wheel_link: mass 1 -> None
- link fr_wheel_link: mass 8 -> None
- link rl_steering_wheel_link: mass 1 -> None
- link rl_wheel_link: mass 8 -> None
- link rr_steering_wheel_link: mass 1 -> None
- link rr_wheel_link: mass 8 -> None
